Commit message: Add camera to Go2

File: robots/go2_description/xacro/gazebo.xacro (robot description, xacro)
@@ -233,3 +233,48 @@
         <kd  value="1.0"/>
     </gazebo>
+    <!-- 深度相机传感器配置 -->
+    <gazebo reference="camera_link">
+    <material>Gazebo/Black</material>
+    <sensor type="depth" name="camera_sensor">
+        <update_rate>10.0</update_rate>
+        <camera name="camera">
+        <horizontal_fov>1.1693706</horizontal_fov> <!-- 67 deg -->
+        <image>
+            <width>480</width>
+            <height>480</height>
+            <format>R8G8B8</format>
+        </image>
+        <depth_camera>
+            <output>depths</output>
+        </depth_camera>
+        <clip>
+            <near>0.02</near>
+            <far>5.0</far>
+        </clip>
+        <noise>
+            <type>gaussian</type>
+            <mean>0.0</mean>
+            <stddev>0.007</stddev>
+        </noise>
+        </camera>
+        <plugin name="camera_controller" filename="libgazebo_ros_openni_kinect.so">
+        <alwaysOn>true</alwaysOn>
+        <updateRate>30.0</updateRate>
+        <cameraName>camera</cameraName>
+        <imageTopicName>rgb/image_raw</imageTopicName>
+        <cameraInfoTopicName>rgb/camera_info</cameraInfoTopicName>
+        <depthImageTopicName>depth/image_raw</depthImageTopicName>
+        <depthImageInfoTopicName>depth/camera_info</depthImageInfoTopicName>
+        <pointCloudTopicName>depth/points</pointCloudTopicName>
+        <frameName>camera_optical_frame</frameName>
+        <pointCloudCutoff>0.1</pointCloudCutoff>
+        <pointCloudCutoffMax>5.0</pointCloudCutoffMax>
+        <distortionK1>0.0</distortionK1>
+        <distortionK2>0.0</distortionK2>
+        <distortionK3>0.0</distortionK3>
+        <distortionT1>0.0</distortionT1>
+        <distortionT2>0.0</distortionT2>
+        </plugin>
+    </sensor>
+    </gazebo>
 </robot>

File: robots/go2_description/xacro/robot.xacro (robot description, xacro)
@@ -118,3 +118,40 @@
     <xacro:leg name="RR" mirror="-1" mirror_dae="False"  front_hind="-1" front_hind_dae="False" />
     <xacro:leg name="RL" mirror="1"  mirror_dae="True"   front_hind="-1" front_hind_dae="False" />
+    <!-- 相机链接 -->
+    <link name="camera_link">
+    <inertial>
+        <origin xyz="0 0 0" rpy="0 0 0"/>
+        <mass value="0.1"/>
+        <inertia ixx="0.001" ixy="0" ixz="0" iyy="0.001" iyz="0" izz="0.001"/>
+    </inertial>
+    <visual>
+        <origin xyz="0 0 0" rpy="0 0 0"/>
+        <geometry>
+        <box size="0.03 0.06 0.03"/>
+        </geometry>
+        <material name="">
+        <color rgba="0.1 0.1 0.1 1"/>
+        </material>
+    </visual>
+    <collision>
+        <origin xyz="0 0 0" rpy="0 0 0"/>
+        <geometry>
+        <box size="0.03 0.03 0.03"/>
+        </geometry>
+    </collision>
+    </link>
+    <!-- 相机关节 - 38度pitch向下倾斜 -->
+    <joint name="camera_joint" type="fixed">
+    <origin xyz="0.35 0.0 0.1" rpy="0 0.663225 0"/> <!-- 0.523599 rad = 30度；0.663225 rad = 38度 -->
+    <parent link="trunk"/>
+    <child link="camera_link"/>
+    </joint>
+    <!-- 相机光学框架 -->
+    <link name="camera_optical_frame">
+    </link>
+    <joint name="camera_optical_joint" type="fixed">
+    <origin xyz="0 0 0" rpy="-1.5707963268 0 -1.5707963268"/> <!-- 旋转调整为光学坐标系 -->
+    <parent link="camera_link"/>
+    <child link="camera_optical_frame"/>
+    </joint>
 </robot>
